File: lazer_tanks_r1/lazer_tanks_r1.sch (KiCad schematic (older format))
At the start: 60 parts, among them J1 Screw_Terminal_01x02, J2 Conn_01x19, J3 Conn_01x19, J4 Conn_01x03_Female, J5 Screw_Terminal_01x02, J6 Screw_Terminal_01x02, J7 Conn_01x03_Female, U1 DMP3056, U2 DMG4822, U3 BQ2961, U4 ESP32-DEVKITC-32D, U5 INA300, U6 DMG4822, U7 TPS565208DDCR, U8 L293DD, U9 TPS565208DDCR

Commit message: Revised schematic to simplify circuit operation
Parts:
- removed BT1, BT2: 3.3V, symbol Device:Battery_Cell
- removed C1, C2, C3: 0.1u, Capacitor_SMD:C_0603_1608Metric_Pad1.05x0.95mm_HandSolder, symbol Device:C
- removed C4: 0.47u, Capacitor_SMD:C_0603_1608Metric_Pad1.05x0.95mm_HandSolder, symbol Device:C
- removed R1, R2: 0, Resistor_SMD:R_0603_1608Metric_Pad1.05x0.95mm_HandSolder, symbol Device:R
- removed R10: 10k, Resistor_SMD:R_0603_1608Metric_Pad1.05x0.95mm_HandSolder, symbol Device:R
- removed R11: 10m, Resistor_SMD:R_1206_3216Metric_Pad1.42x1.75mm_HandSolder, symbol Device:R
- removed R3: 100k, Resistor_SMD:R_0603_1608Metric_Pad1.05x0.95mm_HandSolder, symbol Device:R
- removed R4: 100, Resistor_SMD:R_0603_1608Metric_Pad1.05x0.95mm_HandSolder, symbol Device:R
- removed R6: 1k, Resistor_SMD:R_0603_1608Metric_Pad1.05x0.95mm_HandSolder, symbol Device:R
- removed U1: DMP3056, symbol oraLIB:DMP3056
- removed U2, U6: DMG4822, symbol oraLIB:DMG4822
- removed U3: BQ2961, symbol oraLIB:BQ2961
- removed U5: INA300, symbol oraLIB:INA300
- added F1: Fuse, symbol Device:Fuse
- added J1, J2: Conn_01x02, Connector_JST:JST_EH_B2B-EH-A_1x02_P2.50mm_Vertical, symbol Connector_Generic:Conn_01x02
- added J8, J9: Conn_01x02_Female, symbol Connector:Conn_01x02_Female
- added R7: 0, Resistor_SMD:R_0603_1608Metric_Pad1.05x0.95mm_HandSolder, symbol Device:R
- added SW1: SW_SPST, symbol Switch:SW_SPST
- added U5, U6: DMP3056, symbol oraLIB:DMP3056
- R12: value 100k -> 100
- R13: value 3M -> 100
- R8: value 1k -> 33.2k
- R9: value 5 -> 10k
- renumbered C8 to C1, C20 to C10, C5 to C11, C14 to C12, C10 to C13, C17 to C14, C6 to C15, C7 to C16, C15 to C2, C9 to C3, C16 to C4, C11 to C5, C18 to C6, C12 to C7, C19 to C8, C13 to C9, J7 to J10, J4 to J11, J2 to J3, J3 to J4, J1 to J7, R16 to R1, R5 to R10, R7 to R11, R19 to R2, R14 to R3, R17 to R4, R15 to R5, R18 to R6, U7 to U1, U9 to U2, U8 to U3
Connections:
- net +5V: now also U5.1 (S1), U5.3 (S2), U6.1 (S1), U6.3 (S2)
- net +BATT: now also R7.2, SW1.1 (A)
- net IO2: now also R13.1
- net IO35: now also R8.1, R9.2
- net IO4: now also R12.1
- net at R8.2: now also R7.1
- net -BATT: now reaches R9.1
- net -BATT: now also BZ1.2 (+), C1.2, C10.1, C15.2, C16.1, C2.2, C3.2, C4.2, C5.1, C6.1, C7.1, C8.1, C9.1, J10.3 (Pin_3), J11.3 (Pin_3), J3.6 (Pin_6), J4.13 (Pin_13), J4.19 (Pin_19), J7.2 (Pin_2), R1.1, R2.1, U1.1 (GND), U2.1 (GND), U3.14 (GND), U3.15 (GND), U3.16 (GND), U3.17 (GND), U3.4 (GND), U3.5 (GND), U3.6 (GND), U3.7 (GND), U4.14 (GND1), U4.20 (GND3), U4.26 (GND2), J1.2 (Pin_2), J2.2 (Pin_2), J8.2 (Pin_2), J9.2 (Pin_2)
- net at R13.2: now also U6.4 (G2)
- net at R12.2: now also U6.2 (G1)
- net at R10.2: now also U5.2 (G1)
- net at R11.2: now also U5.4 (G2)
- net at BZ1.1 (-): now also U5.5 (D2), U5.6 (D2)
- net at J7.1 (Pin_1): now also U5.7 (D1), U5.8 (D1)
- removed net GND: BZ1.2 (+), C1.2, C10.1, C15.2, C16.1, C2.2, C3.2, C4.2, C5.1, C6.1, C7.1, C8.1, C9.1, J10.3 (Pin_3), J11.3 (Pin_3), J3.6 (Pin_6), J4.13 (Pin_13), J4.19 (Pin_19), J7.2 (Pin_2), R1.1, R12.1, R13.1, R2.1, U1.1 (GND), U2.1 (GND), U3.14 (GND), U3.15 (GND), U3.16 (GND), U3.17 (GND), U3.4 (GND), U3.5 (GND), U3.6 (GND), U3.7 (GND), U4.14 (GND1), U4.20 (GND3), U4.26 (GND2)
- new net: F1.1, J1.1 (Pin_1), J2.1 (Pin_1)
- new net: F1.2, SW1.2 (B)
- new net: J8.1 (Pin_1), U6.7 (D1), U6.8 (D1)
- new net: J9.1 (Pin_1), U6.5 (D2), U6.6 (D2)
- no-connect marks 5 -> 0
Other:
- note added: "5V Control for IR LED"
- note added: "5V Control for Laser Diode and Buzzer"
- note added: "Battery Sensing Circuit"
- note added: "IR Receiver Header"
- note added: "Parallel Power Input from Batteries"
- note removed: "3V3 Control for Laser Diode and Buzzer"
- note removed: "Battery Protection Circuit"
- note removed: "IR LED Header"
- moved on the sheet: C1, C10, C11, C12, C13, C14, C2, C3, C4, C5, C6, C7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

Commit message: Finalized nearly all footprints
Parts:
- J8, J9: footprint (none) -> Connector_PinHeader_2.54mm:PinHeader_1x02_P2.54mm_Vertical
- U1, U2: footprint (none) -> Package_TO_SOT_SMD:TSOT-23-6_HandSoldering
- U3: footprint (none) -> Package_SO:SO-20_12.8x7.5mm_P1.27mm
- U5, U6: footprint (none) -> Package_SO:SO-8_3.9x4.9mm_P1.27mm
Changed lines of the file:
@@
 F 0 "U1" H 3300 4065 50  0000 C CNN
 F 1 "TPS565208DDCR" H 3300 3974 50  0000 C CNN
-F 2 "" H 3300 3550 50  0001 C CNN
+F 2 "Package_TO_SOT_SMD:TSOT-23-6_HandSoldering" H 3300 3550 50  0001 C CNN
 F 3 "" H 3300 3550 50  0001 C CNN
 	1    3300 3550
@@
 F 0 "U3" H 9250 10150 50  0000 C CNN
 F 1 "L293DD" H 8400 10150 50  0000 C CNN
-F 2 "" H 9000 9850 50  0001 C CNN
+F 2 "Package_SO:SO-20_12.8x7.5mm_P1.27mm" H 9000 9850 50  0001 C CNN
 F 3 "" H 9000 9850 50  0001 C CNN
 	1    8850 8550
@@
 F 0 "U2" H 3350 6465 50  0000 C CNN
 F 1 "TPS565208DDCR" H 3350 6374 50  0000 C CNN
-F 2 "" H 3350 5950 50  0001 C CNN
+F 2 "Package_TO_SOT_SMD:TSOT-23-6_HandSoldering" H 3350 5950 50  0001 C CNN
 F 3 "" H 3350 5950 50  0001 C CNN
 	1    3350 5950
@@
 F 0 "J8" H 14928 2976 50  0000 L CNN
 F 1 "Conn_01x02_Female" H 14928 2885 50  0000 L CNN
-F 2 "" H 14900 3000 50  0001 C CNN
+F 2 "Connector_PinHeader_2.54mm:PinHeader_1x02_P2.54mm_Vertical" H 14900 3000 50  0001 C CNN
 F 3 "~" H 14900 3000 50  0001 C CNN
 	1    14900 3000
@@
 F 0 "J9" H 14928 3426 50  0000 L CNN
 F 1 "Conn_01x02_Female" H 14928 3335 50  0000 L CNN
-F 2 "" H 14900 3450 50  0001 C CNN
+F 2 "Connector_PinHeader_2.54mm:PinHeader_1x02_P2.54mm_Vertical" H 14900 3450 50  0001 C CNN
 F 3 "~" H 14900 3450 50  0001 C CNN
 	1    14900 3450
@@
 F 0 "U5" H 13500 2265 50  0000 C CNN
 F 1 "DMP3056" H 13500 2174 50  0000 C CNN
-F 2 "" H 13900 1750 50  0001 C CNN
+F 2 "Package_SO:SO-8_3.9x4.9mm_P1.27mm" H 13900 1750 50  0001 C CNN
 F 3 "" H 13900 1750 50  0001 C CNN
 	1    13500 1750
@@
 F 0 "U6" H 13550 3765 50  0000 C CNN
 F 1 "DMP3056" H 13550 3674 50  0000 C CNN
-F 2 "" H 13950 3250 50  0001 C CNN
+F 2 "Package_SO:SO-8_3.9x4.9mm_P1.27mm" H 13950 3250 50  0001 C CNN
 F 3 "" H 13950 3250 50  0001 C CNN
 	1    13550 3250
