File: lazer_tanks_r1/lazer_tanks_r1.sch (KiCad schematic (older format))
At the start: 52 parts, among them J1 Conn_01x02, J10 Conn_01x03_Female, J11 Conn_01x03_Female, J2 Conn_01x02, J3 Conn_01x19, J4 Conn_01x19, J5 Screw_Terminal_01x02, J6 Screw_Terminal_01x02, J7 Screw_Terminal_01x02, J8 Conn_01x02_Female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

Commit message: Making second version of board with integrated ESP32
Parts:
- removed U5, U6: DMP3056, Package_SO:SO-8_3.9x4.9mm_P1.27mm, symbol oraLIB:DMP3056
- added C17: 0.1u, Capacitor_SMD:C_0603_1608Metric_Pad1.05x0.95mm_HandSolder, symbol Device:C
- added D1: D, symbol Device:D
- added R14: 100k, Resistor_SMD:R_0603_1608Metric_Pad1.05x0.95mm_HandSolder, symbol Device:R
- added R15, R16, R17, R18: 10k, Resistor_SMD:R_0603_1608Metric_Pad1.05x0.95mm_HandSolder, symbol Device:R
- added U5, U6: DMG4822, symbol oraLIB:DMG4822
- R10, R11, R12, R13: value 100 -> 1k
- gave numbers to parts that had none: 2
Connections:
- net +5V: now also BZ1.1 (-), J7.1 (Pin_1), J8.1 (Pin_1), J9.1 (Pin_1), D1.1 (K)
- net +BATT: now also U7.5 (D2), U7.6 (D2), U7.7 (D1), U7.8 (D1); no longer F1.2
- net -BATT: now also SW1.2 (B), C17.1, R15.2, R16.2, R17.2, R18.2, U5.1 (S1), U5.3 (S2), U6.1 (S1), U6.3 (S2); no longer BZ1.2 (+), J7.2 (Pin_2), J8.2 (Pin_2), J9.2 (Pin_2)
- net IO35: now also C17.2
- net at R10.2: now also R17.1, U5.2 (G1)
- net at R11.2: now also R15.1, U5.4 (G2)
- net at J1.1 (Pin_1), J2.1 (Pin_1): now also F1.1; no longer U7.7 (D1), U7.8 (D1)
- net at SW1.1 (A), U7.2 (G1): now also U7.4 (G2), R14.1; no longer F1.1, U7.1 (S1)
- net at R12.2: now also R18.1, U6.2 (G1)
- net at R13.2: now also R16.1, U6.4 (G2)
- net VBATT: now reaches U7.3 (S2)
- net VBATT: now also F1.2, U7.1 (S1), R14.2
- new net: J7.2 (Pin_2), U5.7 (D1), U5.8 (D1)
- new net: BZ1.2 (+), D1.2 (A), U5.5 (D2), U5.6 (D2)
- new net: J9.2 (Pin_2), U6.5 (D2), U6.6 (D2)
- new net: J8.2 (Pin_2), U6.7 (D1), U6.8 (D1)
Other:
- note removed: "IR Receiver Header"
- moved on the sheet: BZ1, C1, C10, C11, C12, C13, C14, C15, C16, C2, C3, C4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
