File: laser_tanks_r2/laser_tanks_r2/laser_tanks_r2.sch (KiCad schematic (older format))
At the start: 100 parts, among them J1 USB_B_Micro, J10 Conn_01x04, J11 Conn_01x02, J12 Conn_01x02, J13 Conn_01x02, J14 Screw_Terminal_01x02, J15 Screw_Terminal_01x02, J2 Conn_01x04, J3 Screw_Terminal_01x02, J4 Screw_Terminal_01x02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

Commit message: Making new real version of board (tank_board)
Parts:
- added R19: 220, symbol Device:R
- BZ1: footprint (none) -> digikey-footprints:Piezo_Transducer_THT_PS1240P02BT
- C1, C10, C13, C14, C18, C19, C23, C24, C25, C28, C4, C5, C6: footprint (none) -> Capacitor_SMD:C_0603_1608Metric_Pad1.05x0.95mm_HandSolder
- C15, C16: footprint (none) -> Capacitor_SMD:C_1206_3216Metric_Pad1.42x1.75mm_HandSolder
- C17, C2, C20, C26, C3, C7: footprint (none) -> Capacitor_SMD:C_0805_2012Metric_Pad1.15x1.40mm_HandSolder
- C21, C22, C27: footprint (none) -> Capacitor_SMD:CP_Elec_6.3x5.4
Connections:
- net -BATT: now also R19.2
- net at J9.2 (Pin_2), R34.1: now also R19.1
Other:
- moved on the sheet: R34
Changed lines of the file:
@@
 $Descr C 22000 17000
 encoding utf-8
-Sheet 1 1
+Sheet 1 2
 Title ""
 Date ""
@@
 F 0 "C2" H 1515 1896 50  0000 L CNN
 F 1 "10u" H 1515 1805 50  0000 L CNN
-F 2 "" H 1438 1700 50  0001 C CNN
+F 2 "Capacitor_SMD:C_0805_2012Metric_Pad1.15x1.40mm_HandSolder" H 1438 1700 50  0001 C CNN
 F 3 "~" H 1400 1850 50  0001 C CNN
 	1    1400 1850
@@
 F 0 "C3" H 2865 1796 50  0000 L CNN
 F 1 "10u" H 2865 1705 50  0000 L CNN
-F 2 "" H 2788 1600 50  0001 C CNN
+F 2 "Capacitor_SMD:C_0805_2012Metric_Pad1.15x1.40mm_HandSolder" H 2788 1600 50  0001 C CNN
 F 3 "~" H 2750 1750 50  0001 C CNN
 	1    2750 1750
@@
 F 0 "C5" H 3365 6446 50  0000 L CNN
 F 1 "0.1u" H 3365 6355 50  0000 L CNN
-F 2 "" H 3288 6250 50  0001 C CNN
+F 2 "Capacitor_SMD:C_0603_1608Metric_Pad1.05x0.95mm_HandSolder" H 3288 6250 50  0001 C CNN
 F 3 "~" H 3250 6400 50  0001 C CNN
 	1    3250 6400
@@
 F 0 "C1" H 1365 9946 50  0000 L CNN
 F 1 "0.1u (NC)" H 1365 9855 50  0000 L CNN
-F 2 "" H 1288 9750 50  0001 C CNN
+F 2 "Capacitor_SMD:C_0603_1608Metric_Pad1.05x0.95mm_HandSolder" H 1288 9750 50  0001 C CNN
 F 3 "~" H 1250 9900 50  0001 C CNN
 	1    1250 9900
@@
 F 0 "C4" H 3215 9946 50  0000 L CNN
 F 1 "0.1u" H 3215 9855 50  0000 L CNN
-F 2 "" H 3138 9750 50  0001 C CNN
+F 2 "Capacitor_SMD:C_0603_1608Metric_Pad1.05x0.95mm_HandSolder" H 3138 9750 50  0001 C CNN
 F 3 "~" H 3100 9900 50  0001 C CNN
 	1    3100 9900
@@
 F 0 "C7" H 5965 1296 50  0000 L CNN
 F 1 "10u" H 5965 1205 50  0000 L CNN
-F 2 "" H 5888 1100 50  0001 C CNN
+F 2 "Capacitor_SMD:C_0805_2012Metric_Pad1.15x1.40mm_HandSolder" H 5888 1100 50  0001 C CNN
 F 3 "~" H 5850 1250 50  0001 C CNN
 	1    5850 1250
@@
 F 0 "C10" H 6365 1296 50  0000 L CNN
 F 1 "0.1u" H 6365 1205 50  0000 L CNN
-F 2 "" H 6288 1100 50  0001 C CNN
+F 2 "Capacitor_SMD:C_0603_1608Metric_Pad1.05x0.95mm_HandSolder" H 6288 1100 50  0001 C CNN
 F 3 "~" H 6250 1250 50  0001 C CNN
 	1    6250 1250
@@
 F 0 "C6" H 5265 3796 50  0000 L CNN
 F 1 "0.1u" H 5265 3705 50  0000 L CNN
-F 2 "" H 5188 3600 50  0001 C CNN
+F 2 "Capacitor_SMD:C_0603_1608Metric_Pad1.05x0.95mm_HandSolder" H 5188 3600 50  0001 C CNN
 F 3 "~" H 5150 3750 50  0001 C CNN
 	1    5150 3750
@@
 F 0 "C24" V 10898 1100 50  0000 C CNN
 F 1 "0.1u" V 10989 1100 50  0000 C CNN
-F 2 "" H 11188 950 50  0001 C CNN
+F 2 "Capacitor_SMD:C_0603_1608Metric_Pad1.05x0.95mm_HandSolder" H 11188 950 50  0001 C CNN
 F 3 "~" H 11150 1100 50  0001 C CNN
 	1    11150 1100
@@
 F 0 "C26" H 12715 2296 50  0000 L CNN
 F 1 "C" H 12715 2205 50  0000 L CNN
-F 2 "" H 12638 2100 50  0001 C CNN
+F 2 "Capacitor_SMD:C_0805_2012Metric_Pad1.15x1.40mm_HandSolder" H 12638 2100 50  0001 C CNN
 F 3 "~" H 12600 2250 50  0001 C CNN
 	1    12600 2250
@@
 F 0 "C16" H 9885 2054 50  0000 R CNN
 F 1 "22u" H 9885 2145 50  0000 R CNN
-F 2 "" H 10038 1950 50  0001 C CNN
+F 2 "Capacitor_SMD:C_1206_3216Metric_Pad1.42x1.75mm_HandSolder" H 10038 1950 50  0001 C CNN
 F 3 "~" H 10000 2100 50  0001 C CNN
 	1    10000 2100
@@
 F 0 "C15" H 9635 2054 50  0000 R CNN
 F 1 "22u" H 9635 2145 50  0000 R CNN
-F 2 "" H 9788 1950 50  0001 C CNN
+F 2 "Capacitor_SMD:C_1206_3216Metric_Pad1.42x1.75mm_HandSolder" H 9788 1950 50  0001 C CNN
 F 3 "~" H 9750 2100 50  0001 C CNN
 	1    9750 2100
@@
 F 0 "C17" H 10400 2450 50  0000 R CNN
 F 1 "10u" H 10450 2650 50  0000 R CNN
-F 2 "" H 10288 2400 50  0001 C CNN
+F 2 "Capacitor_SMD:C_0805_2012Metric_Pad1.15x1.40mm_HandSolder" H 10288 2400 50  0001 C CNN
 F 3 "~" H 10250 2550 50  0001 C CNN
 	1    10250 2550
@@
 F 0 "C20" H 10550 2650 50  0000 L CNN
 F 1 "10u" H 10550 2450 50  0000 L CNN
-F 2 "" H 10538 2400 50  0001 C CNN
+F 2 "Capacitor_SMD:C_0805_2012Metric_Pad1.15x1.40mm_HandSolder" H 10538 2400 50  0001 C CNN
 F 3 "~" H 10500 2550 50  0001 C CNN
 	1    10500 2550
@@
 F 0 "C23" H 10800 2650 50  0000 L CNN
 F 1 "0.1u" H 10800 2450 50  0000 L CNN
-F 2 "" H 10788 2400 50  0001 C CNN
+F 2 "Capacitor_SMD:C_0603_1608Metric_Pad1.05x0.95mm_HandSolder" H 10788 2400 50  0001 C CNN
 F 3 "~" H 10750 2550 50  0001 C CNN
 	1    10750 2550
@@
 F 0 "C19" H 10350 5900 50  0000 L CNN
 F 1 "0.1u" H 10350 5700 50  0000 L CNN
-F 2 "" H 10338 5650 50  0001 C CNN
+F 2 "Capacitor_SMD:C_0603_1608Metric_Pad1.05x0.95mm_HandSolder" H 10338 5650 50  0001 C CNN
 F 3 "~" H 10300 5800 50  0001 C CNN
 	1    10300 5800
@@
 F 0 "C22" H 10700 5900 50  0000 L CNN
 F 1 "47u" H 10700 5700 50  0000 L CNN
-F 2 "" H 10688 5650 50  0001 C CNN
+F 2 "Capacitor_SMD:CP_Elec_6.3x5.4" H 10688 5650 50  0001 C CNN
 F 3 "~" H 10650 5800 50  0001 C CNN
 	1    10650 5800
@@
 F 0 "C25" H 12550 5900 50  0000 L CNN
 F 1 "0.1u" H 12550 5700 50  0000 L CNN
-F 2 "" H 12538 5650 50  0001 C CNN
+F 2 "Capacitor_SMD:C_0603_1608Metric_Pad1.05x0.95mm_HandSolder" H 12538 5650 50  0001 C CNN
 F 3 "~" H 12500 5800 50  0001 C CNN
 	1    12500 5800
@@
 F 0 "C27" H 12900 5900 50  0000 L CNN
 F 1 "47u" H 12900 5700 50  0000 L CNN
-F 2 "" H 12888 5650 50  0001 C CNN
+F 2 "Capacitor_SMD:CP_Elec_6.3x5.4" H 12888 5650 50  0001 C CNN
 F 3 "~" H 12850 5800 50  0001 C CNN
 	1    12850 5800
@@
 F 0 "C18" H 10300 7450 50  0000 L CNN
 F 1 "0.1u" H 10300 7250 50  0000 L CNN
-F 2 "" H 10288 7200 50  0001 C CNN
+F 2 "Capacitor_SMD:C_0603_1608Metric_Pad1.05x0.95mm_HandSolder" H 10288 7200 50  0001 C CNN
 F 3 "~" H 10250 7350 50  0001 C CNN
 	1    10250 7350
@@
 F 0 "C21" H 10650 7450 50  0000 L CNN
 F 1 "47u" H 10650 7250 50  0000 L CNN
-F 2 "" H 10638 7200 50  0001 C CNN
+F 2 "Capacitor_SMD:CP_Elec_6.3x5.4" H 10638 7200 50  0001 C CNN
 F 3 "~" H 10600 7350 50  0001 C CNN
 	1    10600 7350
@@
 F 0 "C28" H 16515 9596 50  0000 L CNN
 F 1 "0.1u" H 16515 9505 50  0000 L CNN
-F 2 "" H 16438 9400 50  0001 C CNN
+F 2 "Capacitor_SMD:C_0603_1608Metric_Pad1.05x0.95mm_HandSolder" H 16438 9400 50  0001 C CNN
 F 3 "~" H 16400 9550 50  0001 C CNN
 	1    16400 9550
@@
 F 0 "BZ1" H 16702 6029 50  0000 L CNN
 F 1 "Buzzer" H 16702 5938 50  0000 L CNN
-F 2 "" V 16525 6100 50  0001 C CNN
+F 2 "digikey-footprints:Piezo_Transducer_THT_PS1240P02BT" V 16525 6100 50  0001 C CNN
 F 3 "~" V 16525 6100 50  0001 C CNN
 	1    16550 6000
@@
 	1    0    0    -1
 $EndComp
-$Comp
-L power:GND #PWR046
-U 1 1 60300425
-P 14900 4500
-F 0 "#PWR046" H 14900 4250 50  0001 C CNN
-F 1 "GND" H 14905 4327 50  0000 C CNN
-F 2 "" H 14900 4500 50  0001 C CNN
-F 3 "" H 14900 4500 50  0001 C CNN
-	1    14900 4500
-	1    0    0    -1
-$EndComp
 Wire Wire Line
 	14900 4300 15100 4300
-Wire Wire Line
-	14900 4500 15100 4500
 $Comp
 L Device:R R34
 U 1 1 6030042D
-P 14750 4400
-F 0 "R34" V 14543 4400 50  0000 C CNN
-F 1 "220" V 14634 4400 50  0000 C CNN
-F 2 "" V 14680 4400 50  0001 C CNN
-F 3 "~" H 14750 4400 50  0001 C CNN
-	1    14750 4400
+P 14500 4400
+F 0 "R34" V 14293 4400 50  0000 C CNN
+F 1 "220" V 14384 4400 50  0000 C CNN
+F 2 "" V 14430 4400 50  0001 C CNN
+F 3 "~" H 14500 4400 50  0001 C CNN
+	1    14500 4400
 	0    1    1    0
 $EndComp
 Wire Wire Line
-	15100 4400 14900 4400
-Wire Wire Line
-	14600 4400 14250 4400
-Text Label 14250 4400 0    50   ~ 0
+	15100 4400 14700 4400
+Wire Wire Line
+	14350 4400 14050 4400
+Text Label 14050 4400 0    50   ~ 0
 IO33
 Wire Notes Line width 20 style solid
@@
 F 0 "C13" H 7665 1546 50  0000 L CNN
 F 1 "2.7pF" H 7665 1455 50  0000 L CNN
-F 2 "" H 7588 1350 50  0001 C CNN
+F 2 "Capacitor_SMD:C_0603_1608Metric_Pad1.05x0.95mm_HandSolder" H 7588 1350 50  0001 C CNN
 F 3 "~" H 7550 1500 50  0001 C CNN
 	1    7550 1500
@@
 F 0 "C14" V 7648 1200 50  0000 C CNN
 F 1 "4.7pF" V 7739 1200 50  0000 C CNN
-F 2 "" H 7938 1050 50  0001 C CNN
+F 2 "Capacitor_SMD:C_0603_1608Metric_Pad1.05x0.95mm_HandSolder" H 7938 1050 50  0001 C CNN
 F 3 "~" H 7900 1200 50  0001 C CNN
 	1    7900 1200
@@
 Text Notes 7850 10300 0    50   ~ 0
 Battery Integration Circuitry\n
+$Comp
+L Device:R R19
+U 1 1 5DB1519D
+P 14700 4600
+F 0 "R19" V 14493 4600 50  0000 C CNN
+F 1 "220" V 14584 4600 50  0000 C CNN
+F 2 "" V 14630 4600 50  0001 C CNN
+F 3 "~" H 14700 4600 50  0001 C CNN
+	1    14700 4600
+	1    0    0    -1
+$EndComp
+Wire Wire Line
+	14700 4400 14700 4450
+Connection ~ 14700 4400
+Wire Wire Line
+	14700 4400 14650 4400
+Wire Wire Line
+	14700 4750 14700 4900
+$Comp
+L power:GND #PWR046
+U 1 1 60300425
+P 14900 4900
+F 0 "#PWR046" H 14900 4650 50  0001 C CNN
+F 1 "GND" H 14905 4727 50  0000 C CNN
+F 2 "" H 14900 4900 50  0001 C CNN
+F 3 "" H 14900 4900 50  0001 C CNN
+	1    14900 4900
+	1    0    0    -1
+$EndComp
+Wire Wire Line
+	14900 4900 14900 4500
+Wire Wire Line
+	14900 4500 15100 4500
+Wire Wire Line
+	14700 4900 14900 4900
+Connection ~ 14900 4900
+$Sheet
+S 1300 10600 6800 5500
+U 5DC93F6D
+F0 "ESP32_PICO" 98
+F1 "esp32_pico.sch" 98
+$EndSheet
 $EndSCHEMATC
