File: tank_board/esp32wroom.sch (KiCad schematic (older format))
At the start: 24 parts, among them J1 10103594-0001LF, Q1 MMBT3904-7-F, Q2 MMBT3904-7-F, Q3 FDN340P, U1 FT231XS-U, U2 LDL1117S33R

Commit message: Renamed VCC to VBAT
Connections:
- net VCC renamed VBAT
Changed lines of the file:
@@
 	2850 5500 3250 5500
 Connection ~ 2850 5500
-Wire Wire Line
-	3550 5300 3550 5100
 $Comp
 L dk_Interface-Controllers:FT231XS-U U1
@@
 	1    0    0    -1
 $EndComp
-$Comp
-L power:VCC #PWR?
-U 1 1 5E82B569
-P 3550 5100
-F 0 "#PWR?" H 3550 4950 50  0001 C CNN
-F 1 "VCC" H 3567 5273 50  0000 C CNN
-F 2 "" H 3550 5100 50  0001 C CNN
-F 3 "" H 3550 5100 50  0001 C CNN
-	1    3550 5100
-	1    0    0    -1
-$EndComp
+Wire Wire Line
+	3550 5300 3550 5100
+Wire Wire Line
+	3550 5100 3650 5100
+Text GLabel 3650 5100 2    50   Input ~ 0
+VBAT
 $EndSCHEMATC
